File: Hardware/USB_Tool.sch (KiCad schematic (older format))
At the start: 17 parts, among them J1 USB_B_Micro, J2 CONN_ICSP, P1 LED, U1 MCP2210, U2 PIC18F26K40T, X1 CONN_01X03, Y1 DSC6003JI2A

Commit message: First part done, usb to spi
Parts:
- P1: value LED -> 2V
- R2: value R -> 560R
- R4: value R -> 1k
Changed lines of the file:
@@
 EESchema Schematic File Version 4
+LIBS:USB_Tool-cache
 EELAYER 29 0
 EELAYER END
 $Descr A4 11693 8268
 encoding utf-8
-Sheet 1 1
-Title ""
-Date ""
-Rev ""
-Comp ""
-Comment1 ""
-Comment2 ""
+Sheet 1 2
+Title "USB_Tool"
+Date "2019-04-14"
+Rev "00"
+Comp "EsseivaN"
+Comment1 "Author : Esseiva Nicolas"
+Comment2 "Description here"
 Comment3 ""
 Comment4 ""
@@
 P 4600 1750
 F 0 "R4" H 4531 1704 50  0000 R CNN
-F 1 "R" H 4531 1795 50  0000 R CNN
+F 1 "1k" H 4531 1795 50  0000 R CNN
 F 2 "" V 4530 1750 50  0000 C CNN
 F 3 "" H 4600 1750 50  0000 C CNN
@@
 P 3050 2400
 F 0 "P1" V 2997 2478 60  0000 L CNN
-F 1 "LED" V 3103 2478 60  0000 L CNN
+F 1 "2V" V 3103 2478 60  0000 L CNN
 F 2 "" H 3050 2400 60  0000 C CNN
 F 3 "" H 3050 2400 60  0000 C CNN
@@
 P 3050 2100
 F 0 "R2" H 3120 2146 50  0000 L CNN
-F 1 "R" H 3120 2055 50  0000 L CNN
+F 1 "560R" H 3120 2055 50  0000 L CNN
 F 2 "" V 2980 2100 50  0000 C CNN
 F 3 "" H 3050 2100 50  0000 C CNN

Commit message: update TBD
Parts:
- removed U2: PIC18F26K40T, Housings_SSOP:SSOP-28_5.3x10.2mm_Pitch0.65mm, symbol 0EsseivaN_Lib:PIC18F26K40T
- added C?: 100nF, symbol USB_Tool-rescue:CAPA-0EsseivaN_Lib
- added J?: Extender_1, symbol Connector_Generic:Conn_01x04
- added J?: Extender_2, symbol Connector_Generic:Conn_01x04
- added J?: Extender_3, symbol Connector_Generic:Conn_01x04
- added U?: PIC18F45K40_44, symbol 0EsseivaN_Lib_2:PIC18F45K40_44
- added U?: MRF89XAM8A, symbol 0EsseivaN_Lib_2:MRF89XAM8A
- C1, C3, C5: symbol 0EsseivaN_Lib:CAPA -> USB_Tool-rescue:CAPA-0EsseivaN_Lib
- C2, C4: symbol 0EsseivaN_Lib:CAPA_P -> USB_Tool-rescue:CAPA_P-0EsseivaN_Lib
- F1: symbol 0EsseivaN_Lib:Fuse -> USB_Tool-rescue:Fuse-0EsseivaN_Lib
- J1: symbol 0EsseivaN_Lib:USB_B_Micro -> USB_Tool-rescue:USB_B_Micro-0EsseivaN_Lib
- J2: symbol 0EsseivaN_Lib:CONN_ICSP -> USB_Tool-rescue:CONN_ICSP-0EsseivaN_Lib
- P1: symbol 0EsseivaN_Lib:LED -> USB_Tool-rescue:LED-0EsseivaN_Lib
- R1, R2, R3, R4: symbol 0EsseivaN_Lib:R -> USB_Tool-rescue:R-0EsseivaN_Lib
- U1: symbol 0EsseivaN_Lib:MCP2210 -> USB_Tool-rescue:MCP2210-0EsseivaN_Lib
- X1: symbol 0EsseivaN_Lib:CONN_01X03 -> USB_Tool-rescue:CONN_01X03-0EsseivaN_Lib
- Y1: symbol 0EsseivaN_Lib:DSC6003JI2A -> USB_Tool-rescue:DSC6003JI2A-0EsseivaN_Lib
Connections:
- net labels added: BRA, BRR, GND-0EsseivaN_Lib, ICSPCLK, ICSPDAT, SCL, SDA, VPP, ~CS~_RF
- wire segments 88 -> 143
- no-connect marks 23 -> 9
Other:
- note added: "I2C"
- note added: "MASTER #1 SPI"
- note added: "MASTER #2 SPI"
- note added: "SLAVE SPI"
- note added: "USB IO"

Commit message: added rf module
3v3 ldo
switch power
Parts:
- removed J?: Extender_1, symbol Connector_Generic:Conn_01x04
- removed J?: Extender_2, symbol Connector_Generic:Conn_01x04
- removed J?: Extender_3, symbol Connector_Generic:Conn_01x04
- removed X1: CONN_01X03, symbol USB_Tool-rescue:CONN_01X03-0EsseivaN_Lib
- added C?: 4.7uF, symbol USB_Tool-rescue:CAPA-0EsseivaN_Lib
- added C?: 1uF, symbol USB_Tool-rescue:CAPA_P-0EsseivaN_Lib
- added J?: Extender 1, symbol Connector_Generic:Conn_01x05
- added J?: Extender 2, symbol Connector_Generic:Conn_01x05
- added J?: Extender 3, symbol Connector_Generic:Conn_01x05
- added SW?: SW_2TO1, symbol 0EsseivaN_Lib_2:SW_2TO1
- added U?: NCP114, symbol 0EsseivaN_Lib_2:NCP114
Connections:
- net labels added: IRQ0, IRQ1, RESET_RF, RESET_USB, ~CSCON, ~CSDAT
- net labels removed: V_BUS, V_ICSP, ~CS~_RF
- wire segments 143 -> 186
Other:
- note added: "12MHz\noscillator"
- note added: "5V TO 3V3 LDO"
- note removed: "I2C"
- note removed: "MASTER #1 SPI"
- note removed: "MASTER #2 SPI"
- note removed: "SLAVE SPI"
- note removed: "USB IO"

Commit message: Updated TBD
Parts:
- removed U1: MCP2210, Housings_SSOP:SSOP-20_5.3x7.2mm_Pitch0.65mm, symbol USB_Tool-rescue:MCP2210-0EsseivaN_Lib
- added R?: 1k, symbol USB_Tool-rescue:R-0EsseivaN_Lib
- added U?: MCP2210, Housings_SSOP:SSOP-20_5.3x7.2mm_Pitch0.65mm, symbol 0EsseivaN_Lib_2:MCP2210
Connections:
- wire segments 186 -> 208
- no-connect marks 9 -> 12
Other:
- note added: "Ajouter led"
- note added: "USB to SPI"

Commit message: Merged libraries and fixed errors
Parts:
- C1, C3, C5, C? (x2): symbol USB_Tool-rescue:CAPA-0EsseivaN_Lib -> 0EsseivaN_Lib:CAPA
- C2, C4, C?: symbol USB_Tool-rescue:CAPA_P-0EsseivaN_Lib -> 0EsseivaN_Lib:CAPA_P
- F1: symbol USB_Tool-rescue:Fuse-0EsseivaN_Lib -> 0EsseivaN_Lib:Fuse
- J1: symbol USB_Tool-rescue:USB_B_Micro-0EsseivaN_Lib -> 0EsseivaN_Lib:USB_B_Micro
- J2: symbol USB_Tool-rescue:CONN_ICSP-0EsseivaN_Lib -> 0EsseivaN_Lib:CONN_ICSP
- P1: symbol USB_Tool-rescue:LED-0EsseivaN_Lib -> 0EsseivaN_Lib:LED
- R1, R2, R3, R4, R?: symbol USB_Tool-rescue:R-0EsseivaN_Lib -> 0EsseivaN_Lib:R
- SW?: symbol 0EsseivaN_Lib_2:SW_2TO1 -> 0EsseivaN_Lib:SW_2TO1
- U?: symbol 0EsseivaN_Lib_2:PIC18F45K40_44 -> 0EsseivaN_Lib:PIC18F45K40_44
- U?: symbol 0EsseivaN_Lib_2:MCP2210 -> 0EsseivaN_Lib:MCP2210
- U?: symbol 0EsseivaN_Lib_2:NCP114 -> 0EsseivaN_Lib:NCP114
- U?: symbol 0EsseivaN_Lib_2:MRF89XAM8A -> 0EsseivaN_Lib:MRF89XAM8A
- Y1: symbol USB_Tool-rescue:DSC6003JI2A-0EsseivaN_Lib -> 0EsseivaN_Lib:DSC6003JI2A
Connections:
- net labels removed: GND-0EsseivaN_Lib
- wire segments 208 -> 188
- no-connect marks 12 -> 9
Changed lines of the file:
@@
 $EndDescr
 $Comp
-L USB_Tool-rescue:USB_B_Micro-0EsseivaN_Lib J1
+L 0EsseivaN_Lib:USB_B_Micro J1
 U 1 1 5CB4CD34
 P 1200 1000
@@
 	1    0    0    -1
 $EndComp
-$Comp
-L USB_Tool-rescue:5V-0EsseivaN_Lib #PWR0101
-U 1 1 5CB5CED0
-P 11050 -2150
-F 0 "#PWR0101" H 11050 -2300 50  0001 C CNN
-F 1 "5V" H 11067 -1980 45  0000 C CNN
-F 2 "" H 11050 -2150 50  0000 C CNN
-F 3 "" H 11050 -2150 50  0000 C CNN
-	1    11050 -2150
-	1    0    0    -1
-$EndComp
-Wire Wire Line
-	11150 -1450 11050 -1450
-Wire Wire Line
-	11050 -1450 11050 -2100
-Wire Wire Line
-	10950 -2000 10950 -2100
-Wire Wire Line
-	10950 -2100 11050 -2100
-Connection ~ 11050 -2100
-Wire Wire Line
-	11050 -2100 11050 -2150
-Wire Wire Line
-	10950 -1600 10950 -1150
-Wire Wire Line
-	10950 -1150 11150 -1150
 Text GLabel 1800 1000 2    50   BiDi ~ 0
 D+
@@
 D-
 $Comp
-L USB_Tool-rescue:CAPA-0EsseivaN_Lib C5
+L 0EsseivaN_Lib:CAPA C5
 U 1 1 5CB6B8DF
 P 4200 1850
@@
 $EndComp
 $Comp
-L USB_Tool-rescue:GND-0EsseivaN_Lib #PWR0102
+L 0EsseivaN_Lib:GND #PWR0102
 U 1 1 5CB6DCDC
 P 4200 2000
@@
 $EndComp
 $Comp
-L USB_Tool-rescue:GND-0EsseivaN_Lib #PWR0106
+L 0EsseivaN_Lib:GND #PWR0106
 U 1 1 5CB76392
 P 6300 2800
@@
 	6300 2800 6300 2750
 $Comp
-L USB_Tool-rescue:3V3-0EsseivaN_Lib #PWR0107
+L 0EsseivaN_Lib:3V3 #PWR0107
 U 1 1 5CB77422
 P 5500 1900
@@
 $EndComp
 $Comp
-L USB_Tool-rescue:3V3-0EsseivaN_Lib #PWR0109
+L 0EsseivaN_Lib:3V3 #PWR0109
 U 1 1 5CB794E8
 P 6300 2050
@@
 	-1   0    0    -1
 $EndComp
-NoConn ~ 11150 -1250
 NoConn ~ 1500 1200
 $Comp
-L USB_Tool-rescue:GND-0EsseivaN_Lib #PWR0110
+L 0EsseivaN_Lib:GND #PWR0110
 U 1 1 5CB7DD0D
 P 1200 1900
@@
 $EndComp
 $Comp
-L USB_Tool-rescue:R-0EsseivaN_Lib R1
+L 0EsseivaN_Lib:R R1
 U 1 1 5CB7FC9D
 P 1100 1600
@@
 	1200 1900 1200 1850
 $Comp
-L USB_Tool-rescue:CAPA-0EsseivaN_Lib C1
+L 0EsseivaN_Lib:CAPA C1
 U 1 1 5CB83229
 P 850 1600
@@
 Connection ~ 1100 1850
 $Comp
-L USB_Tool-rescue:CAPA-0EsseivaN_Lib C3
+L 0EsseivaN_Lib:CAPA C3
 U 1 1 5CB88B5C
 P 5700 2100
@@
 	5500 1950 5500 2550
 $Comp
-L USB_Tool-rescue:GND-0EsseivaN_Lib #PWR0111
+L 0EsseivaN_Lib:GND #PWR0111
 U 1 1 5CB8C722
 P 5700 2200
@@
 $EndComp
 $Comp
-L USB_Tool-rescue:R-0EsseivaN_Lib R4
+L 0EsseivaN_Lib:R R4
 U 1 1 5CB6108A
 P 5050 2000
@@
 $EndComp
 $Comp
-L USB_Tool-rescue:R-0EsseivaN_Lib R3
+L 0EsseivaN_Lib:R R3
 U 1 1 5CB8D825
 P 6300 2300
@@
 	6300 2500 6300 2550
 $Comp
-L USB_Tool-rescue:CAPA_P-0EsseivaN_Lib C4
+L 0EsseivaN_Lib:CAPA_P C4
 U 1 1 5CB8DCBC
 P 3850 3700
@@
 	0    1    1    0
 $EndComp
-Wire Wire Line
-	11200 -2050 11200 -2100
-Wire Wire Line
-	11200 -2100 11050 -2100
-$Comp
-L USB_Tool-rescue:GND-0EsseivaN_Lib #PWR0112
-U 1 1 5CB918FF
-P 11200 -1800
-F 0 "#PWR0112" H 11200 -2100 50  0001 C CNN
-F 1 "GND" H 11200 -2000 50  0001 C CNN
-F 2 "" H 11200 -1800 50  0000 C CNN
-F 3 "" H 11200 -1800 50  0000 C CNN
-	1    11200 -1800
-	1    0    0    -1
-$EndComp
-Wire Wire Line
-	11200 -1800 11200 -1850
-Wire Wire Line
-	11150 -650 10650 -650
-$Comp
-L USB_Tool-rescue:CONN_ICSP-0EsseivaN_Lib J2
+$Comp
+L 0EsseivaN_Lib:CONN_ICSP J2
 U 1 1 5CBB0674
 P 800 2400
@@
 $EndComp
 $Comp
-L USB_Tool-rescue:GND-0EsseivaN_Lib #PWR0113
+L 0EsseivaN_Lib:GND #PWR0113
 U 1 1 5CBC32A7
 P 1200 2700
@@
 	3450 900  3650 900
 $Comp
-L USB_Tool-rescue:Fuse-0EsseivaN_Lib F1
+L 0EsseivaN_Lib:Fuse F1
 U 1 1 5CB94C5C
 P 3250 900
@@
 	3650 950  3650 900
 $Comp
-L USB_Tool-rescue:GND-0EsseivaN_Lib #PWR0114
+L 0EsseivaN_Lib:GND #PWR0114
 U 1 1 5CB90A85
 P 3650 1400
@@
 $EndComp
 $Comp
-L USB_Tool-rescue:CAPA_P-0EsseivaN_Lib C2
+L 0EsseivaN_Lib:CAPA_P C2
 U 1 1 5CB87644
 P 3650 1050
@@
 	3650 850  3650 900
 $Comp
-L USB_Tool-rescue:5V-0EsseivaN_Lib #PWR0115
+L 0EsseivaN_Lib:5V #PWR0115
 U 1 1 5CB6770D
 P 3650 850
@@
 Connection ~ 1200 1850
 $Comp
-L USB_Tool-rescue:LED-0EsseivaN_Lib P1
+L 0EsseivaN_Lib:LED P1
 U 1 1 5CBEA842
 P 3600 2350
@@
 $EndComp
 $Comp
-L USB_Tool-rescue:R-0EsseivaN_Lib R2
+L 0EsseivaN_Lib:R R2
 U 1 1 5CBEC042
 P 3600 2050
@@
 	1    0    0    -1
 $EndComp
-Wire Wire Line
-	11150 -750 9400 -750
-$Comp
-L USB_Tool-rescue:5V-0EsseivaN_Lib #PWR0116
+$Comp
+L 0EsseivaN_Lib:5V #PWR0116
 U 1 1 5CBEEF46
 P 3600 1850
@@
 	1    0    0    -1
 $EndComp
-Wire Wire Line
-	11150 -850 10600 -850
 Text Label 3950 2950 2    50   ~ 0
 ~USBCFG
 Text Label 3950 2650 2    50   ~ 0
 ~SSPND
-Wire Wire Line
-	11150 -550 10700 -550
 Text Label 3950 2850 2    50   ~ 0
 ~LOWPWR
@@
 Text Label 5050 3450 0    50   ~ 0
 SDI
-NoConn ~ 11150 -1050
-NoConn ~ 11150 -950
 Wire Wire Line
 	6300 2050 6300 2100
@@
 Text Label 5050 3250 0    50   ~ 0
 SCK
-Wire Wire Line
-	10650 -150 10650 -650
 Text Label 6900 3300 2    50   ~ 0
 BRR
@@
 NoConn ~ 7000 5200
 $Comp
-L 0EsseivaN_Lib_2:PIC18F45K40_44 U?
+L 0EsseivaN_Lib:PIC18F45K40_44 U?
 U 1 1 5CB7FF60
 P 7800 4400
@@
 	7800 5950 7800 5900
 $Comp
-L USB_Tool-rescue:GND-0EsseivaN_Lib #PWR?
+L 0EsseivaN_Lib:GND #PWR?
 U 1 1 5CBB7C21
 P 7800 5950
 F 0 "#PWR?" H 7800 5650 50  0001 C CNN
-F 1 "GND-0EsseivaN_Lib" H 7800 5750 50  0001 C CNN
+F 1 "GND" H 7800 5750 50  0001 C CNN
 F 2 "" H 7800 5950 50  0000 C CNN
 F 3 "" H 7800 5950 50  0000 C CNN
@@
 	8200 2800 8200 2750
 $Comp
-L USB_Tool-rescue:GND-0EsseivaN_Lib #PWR?
+L 0EsseivaN_Lib:GND #PWR?
 U 1 1 5CB97922
 P 8200 2800
 F 0 "#PWR?" H 8200 2500 50  0001 C CNN
-F 1 "GND-0EsseivaN_Lib" H 8200 2600 50  0001 C CNN
+F 1 "GND" H 8200 2600 50  0001 C CNN
 F 2 "" H 8200 2800 50  0000 C CNN
 F 3 "" H 8200 2800 50  0000 C CNN
@@
 $EndComp
 $Comp
-L USB_Tool-rescue:CAPA-0EsseivaN_Lib C?
+L 0EsseivaN_Lib:CAPA C?
 U 1 1 5CB96E3E
 P 8200 2650
@@
 Text Label 6900 3500 2    50   ~ 0
 ~USBCFG
-Wire Wire Line
-	10700 -550 10700 -300
-Wire Wire Line
-	10600 -850 10600 -400
 Text Label 6900 3700 2    50   ~ 0
 ~SSPND
@@
 5V
 $Comp
-L USB_Tool-rescue:5V-0EsseivaN_Lib #PWR?
+L 0EsseivaN_Lib:5V #PWR?
 U 1 1 5CC49943
 P 8200 2300
@@
 Connection ~ 8200 2400
 $Comp
-L USB_Tool-rescue:5V-0EsseivaN_Lib #PWR?
+L 0EsseivaN_Lib:5V #PWR?
 U 1 1 5CC4CF73
 P 1200 3000
@@
 	6650 4600 7000 4600
 $Comp
-L 0EsseivaN_Lib_2:MRF89XAM8A U?
+L 0EsseivaN_Lib:MRF89XAM8A U?
 U 1 1 5CCB5FB4
 P 3550 5500
@@
 	3550 6200 3650 6200
 $Comp
-L USB_Tool-rescue:GND-0EsseivaN_Lib #PWR?
+L 0EsseivaN_Lib:GND #PWR?
 U 1 1 5CCD241E
 P 3550 6250
 F 0 "#PWR?" H 3550 5950 50  0001 C CNN
-F 1 "GND-0EsseivaN_Lib" H 3550 6050 50  0001 C CNN
+F 1 "GND" H 3550 6050 50  0001 C CNN
 F 2 "" H 3550 6250 50  0000 C CNN
 F 3 "" H 3550 6250 50  0000 C CNN
@@
 	3550 6200 3550 6250
 $Comp
-L USB_Tool-rescue:3V3-0EsseivaN_Lib #PWR?
+L 0EsseivaN_Lib:3V3 #PWR?
 U 1 1 5CCDE1A2
 P 3550 4750
@@
 $EndComp
 $Comp
-L USB_Tool-rescue:CAPA-0EsseivaN_Lib C?
+L 0EsseivaN_Lib:CAPA C?
 U 1 1 5CB772E2
 P 3950 4900
@@
 	3550 4800 3550 5000
 $Comp
-L USB_Tool-rescue:GND-0EsseivaN_Lib #PWR?
+L 0EsseivaN_Lib:GND #PWR?
 U 1 1 5CB84231
 P 3950 5000
 F 0 "#PWR?" H 3950 4700 50  0001 C CNN
-F 1 "GND-0EsseivaN_Lib" H 3950 4800 50  0001 C CNN
+F 1 "GND" H 3950 4800 50  0001 C CNN
 F 2 "" H 3950 5000 50  0000 C CNN
 F 3 "" H 3950 5000 50  0000 C CNN
@@
 Text Label 6900 4500 2    50   ~ 0
 RESET_USB
-Wire Wire Line
-	10500 -50  10500 -1000
-Wire Wire Line
-	10950 -1000 10950 -1150
-Connection ~ 10950 -1150
 Text Label 6900 4000 2    50   ~ 0
 RESET_RF
@@
 Text Label 3100 5400 2    50   ~ 0
 RESET_RF
-Wire Wire Line
-	10500 -1000 10950 -1000
 Text Notes 5750 2400 0    50   ~ 0
 12MHz\noscillator
 $Comp
-L 0EsseivaN_Lib_2:NCP114 U?
+L 0EsseivaN_Lib:NCP114 U?
 U 1 1 5CC9D2C7
 P 4500 1000
@@
 	4900 1000 5150 1000
 $Comp
-L USB_Tool-rescue:3V3-0EsseivaN_Lib #PWR?
+L 0EsseivaN_Lib:3V3 #PWR?
 U 1 1 5CCD0867
 P 5150 950
@@
 	5150 950  5150 1000
 $Comp
-L USB_Tool-rescue:CAPA_P-0EsseivaN_Lib C?
+L 0EsseivaN_Lib:CAPA_P C?
 U 1 1 5CCD94D7
 P 5150 1150
@@
 	1200 3150 1200 3000
 $Comp
-L USB_Tool-rescue:3V3-0EsseivaN_Lib #PWR?
+L 0EsseivaN_Lib:3V3 #PWR?
 U 1 1 5CD41FD0
 P 1350 3000
@@
 Connection ~ 1400 3550
 $Comp
-L USB_Tool-rescue:GND-0EsseivaN_Lib #PWR?
+L 0EsseivaN_Lib:GND #PWR?
 U 1 1 5CD7F211
 P 1550 3600
@@
 Connection ~ 1400 4300
 $Comp
-L 0EsseivaN_Lib_2:SW_2TO1 SW?
+L 0EsseivaN_Lib:SW_2TO1 SW?
 U 1 1 5CDC9373
 P 2750 900
@@
 SDA
 $Comp
-L USB_Tool-rescue:R-0EsseivaN_Lib R?
+L 0EsseivaN_Lib:R R?
 U 1 1 5CB7D3C5
 P 2700 4550
@@
 	2700 4300 2700 4350
 $Comp
-L USB_Tool-rescue:3V3-0EsseivaN_Lib #PWR?
+L 0EsseivaN_Lib:3V3 #PWR?
 U 1 1 5CB93503
 P 2700 4300
@@
 	2700 4750 2700 4850
 $Comp
-L 0EsseivaN_Lib_2:MCP2210 U?
+L 0EsseivaN_Lib:MCP2210 U?
 U 1 1 5CBE857C
 P 4500 2950
@@
 $EndComp
 $Comp
-L USB_Tool-rescue:DSC6003JI2A-0EsseivaN_Lib Y1
+L 0EsseivaN_Lib:DSC6003JI2A Y1
 U 1 1 5CB74EB9
 P 5900 2650
@@
 Connection ~ 4500 1750
 $Comp
-L USB_Tool-rescue:5V-0EsseivaN_Lib #PWR?
+L 0EsseivaN_Lib:5V #PWR?
 U 1 1 5CE9F6D1
 P 4500 1700
@@
 Connection ~ 6000 4200
 $Comp
-L USB_Tool-rescue:GND-0EsseivaN_Lib #PWR?
+L 0EsseivaN_Lib:GND #PWR?
 U 1 1 5CF8B611
 P 4500 3950

Commit message: TBD
Parts:
- added P2, P3, P4: 2V, symbol 0EsseivaN_Lib:LED
- added R10, R9: 1k, symbol 0EsseivaN_Lib:R
- added R6, R7, R8: 560R, symbol 0EsseivaN_Lib:R
- added X1: CONN_01X07, symbol 0EsseivaN_Lib:CONN_01X07
- added X2, X3: CONN_01X08, symbol 0EsseivaN_Lib:CONN_01X08
- added X4: CONN_01X06, symbol 0EsseivaN_Lib:CONN_01X06
- gave numbers to parts that had none: 12
Connections:
- net labels added: CS, MISO, MOSI
- wire segments 188 -> 266

Commit message: Cleanup and software project created
Parts:
- added R11: 27k, symbol 0EsseivaN_Lib:R
- J3: value Extender 1 -> Extender_I2C_1
- J4: value Extender 2 -> Extender_I2C_2
- J5: value Extender 3 -> Extender_I2C_3
- U4: symbol 0EsseivaN_Lib:PIC18F45K40_44 -> 0EsseivaN_Lib:PIC18F46K40_44
- X1: value CONN_01X07 -> EXTENDER_SPI_1
- X2: value CONN_01X08 -> EXTENDER_IO_1
- X3: value CONN_01X08 -> EXTENDER_IO_2
- X4: value CONN_01X06 -> EXTENDER_IO_3
Connections:
- net GND: now also J2.3 (GND)
- net ICSPCLK: now also J2.5 (ICSPCLK)
- net ICSPDAT: now also J2.4 (ICSPDAT)
- net IRQ0: now also U4.25 (RE0); no longer U4.26 (RE1)
- net IRQ1: now also U4.26 (RE1); no longer U4.25 (RE0)
- net VCC: now also R11.1
- net VPP: now also J2.1 (VPP), R11.2
- net ~CSCON: now also U4.42 (RC4); no longer U4.24 (RA5)
- net ~CSDAT: now also U4.24 (RA5); no longer U4.31 (RA6)
- net ~USBCFG: now also U4.37 (RC3); no longer U4.21 (RA2)
- net LED_0: now reaches P2.2 (Cathode), U4.32 (RC0)
- net LED_1: now reaches P3.2 (Cathode), U4.35 (RC1)
- net LED_2: now reaches P4.2 (Cathode), U4.36 (RC2)
- net D3: now reaches U4.1 (RC7), X2.7 (P7)
- net D8: now reaches U4.2 (RD4), X3.4 (P4)
- net D9: now reaches U4.3 (RD5), X3.5 (P5)
- net DAC1: now reaches X2.3 (P3)
- net DAC1: now also U4.21 (RA2); no longer U4.37 (RC3)
- net D4: now reaches U4.38 (RD0), X2.8 (P8)
- net D5: now reaches U4.39 (RD1), X3.1 (P1)
- net D10: now reaches U4.4 (RD6), X3.6 (P6)
- net D6: now reaches U4.40 (RD2), X3.2 (P2)
- net D7: now reaches U4.41 (RD3), X3.3 (P3)
- net CLK: now reaches X2.4 (P4)
- net CLK: now also U4.31 (RA6); no longer U4.42 (RC4)
- net D1: now reaches U4.43 (RC5), X2.5 (P5)
- net D2: now reaches U4.44 (RC6), X2.6 (P6)
- net D11: now reaches U4.5 (RD7), X3.7 (P7)
- net at J2.2 (VCC): now also SW1.3 (Q2)
- net CS renamed CS_EXT
- no-connect marks 9 -> 12
Other:
- moved on the sheet: C8, J3, J4, J5, R5, X1

Commit message: tbd
Parts:
- added U5: ULN2003, symbol 0EsseivaN_Lib:ULN200x
- F1: value 630mA -> 500mA
- X4: value EXTENDER_IO_3 -> EXTENDER_POWER_1
Connections:
- net GND: now also U5.8 (GND)
- net VCC: now also U5.9 (COM)
- net D10 renamed IP6
- net IP6: now also U5.6 (I6); no longer X3.6 (P6)
- net D11 renamed IP7
- net IP7: now also U5.7 (I7); no longer X3.7 (P7)
- net D5 renamed IP1
- net IP1: now also U5.1 (I1); no longer X3.1 (P1)
- net D6 renamed IP2
- net IP2: now also U5.2 (I2); no longer X3.2 (P2)
- net D7 renamed IP3
- net IP3: now also U5.3 (I3); no longer X3.3 (P3)
- net D8 renamed IP4
- net IP4: now also U5.4 (I4); no longer X3.4 (P4)
- net D9 renamed IP5
- net IP5: now also U5.5 (I5); no longer X3.5 (P5)
- new net P1: U5.16 (O1), X3.1 (P1)
- new net P2: U5.15 (O2), X3.2 (P2)
- new net P3: U5.14 (O3), X3.3 (P3)
- new net P4: U5.13 (O4), X3.4 (P4)
- new net P5: U5.12 (O5), X3.5 (P5)
- new net P6: U5.11 (O6), X3.6 (P6)
- new net P7: U5.10 (O7), X3.7 (P7)
Other:
- note added: "WARNING : Power MCP2210 and\nPIC with same voltages"
- moved on the sheet: C1, C2, C3, C4, C5, C6, C7, C8, F1, J1, J2, J3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
