File: Hardware/USB_Tool.sch (KiCad schematic (older format))
At the start: 40 parts, among them J1 USB_B_Micro, J2 CONN_ICSP, J3 Extender_I2C_1, J4 Extender_I2C_2, J5 Extender_I2C_3, P1 2V, P2 2V, P3 2V, P4 2V, SW1 SW_2TO1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

Commit message: tbd
Parts:
- removed P2, P3, P4: 2V, symbol 0EsseivaN_Lib:LED
- added C9: 100nF, symbol 0EsseivaN_Lib:CAPA
- added P2: 150141M173100, symbol 0EsseivaN_Lib:LED_RGB
- added X5: EXTENDER_COM, symbol 0EsseivaN_Lib:CONN_01X02
- P1: value 2V -> TLMS1000
- R2, R6, R7: value 560R -> 180R
- R8: value 560R -> 270R
- U4: value PIC18F45K40_44 -> PIC18F46K40_44
Connections:
- net 5V: no longer R6.1, R7.1, R8.1, U5.9 (COM)
- net GND: now also C9.2
- net LED_0: now also R6.2
- net LED_1: now also R7.2
- net LED_2: now also R8.2
- new net: P2.4 (GREEN), R7.1
- new net: P2.3 (RED), R8.1
- new net: P2.2 (BLUE), R6.1
- new net COM: C9.1, U5.9 (COM)
Other:
- moved on the sheet: R6, R7, R8
Changed lines of the file:
@@
 U 1 1 5CBEA842
 P 2150 2800
-F 0 "P1" V 2097 2878 60  0000 L CNN
-F 1 "2V" V 2203 2878 60  0000 L CNN
+F 0 "P1" V 2097 2623 60  0000 R CNN
+F 1 "TLMS1000" V 2203 2623 60  0000 R CNN
 F 2 "" H 2150 2800 60  0000 C CNN
 F 3 "" H 2150 2800 60  0000 C CNN
@@
 P 2150 2500
 F 0 "R2" H 2220 2546 50  0000 L CNN
-F 1 "560R" H 2220 2455 50  0000 L CNN
+F 1 "180R" H 2220 2455 50  0000 L CNN
 F 2 "" V 2080 2500 50  0000 C CNN
 F 3 "" H 2150 2500 50  0000 C CNN
@@
 USB to SPI
 $Comp
-L 0EsseivaN_Lib:LED P2
-U 1 1 5CB7DAF4
-P 7550 2300
-F 0 "P2" V 7497 2378 60  0000 L CNN
-F 1 "2V" V 7603 2378 60  0000 L CNN
-F 2 "" H 7550 2300 60  0000 C CNN
-F 3 "" H 7550 2300 60  0000 C CNN
-	1    7550 2300
-	0    1    1    0
-$EndComp
-$Comp
-L 0EsseivaN_Lib:LED P3
-U 1 1 5CB7F24F
-P 7900 2300
-F 0 "P3" V 7847 2378 60  0000 L CNN
-F 1 "2V" V 7953 2378 60  0000 L CNN
-F 2 "" H 7900 2300 60  0000 C CNN
-F 3 "" H 7900 2300 60  0000 C CNN
-	1    7900 2300
-	0    1    1    0
-$EndComp
-$Comp
-L 0EsseivaN_Lib:LED P4
-U 1 1 5CB7F5A3
-P 8250 2300
-F 0 "P4" V 8197 2378 60  0000 L CNN
-F 1 "2V" V 8303 2378 60  0000 L CNN
-F 2 "" H 8250 2300 60  0000 C CNN
-F 3 "" H 8250 2300 60  0000 C CNN
-	1    8250 2300
-	0    1    1    0
-$EndComp
-$Comp
 L 0EsseivaN_Lib:R R7
 U 1 1 5CB7F98F
-P 7900 1950
-F 0 "R7" H 7970 1996 50  0000 L CNN
-F 1 "560R" H 7970 1905 50  0000 L CNN
-F 2 "" V 7830 1950 50  0000 C CNN
-F 3 "" H 7900 1950 50  0000 C CNN
-	1    7900 1950
+P 8000 2200
+F 0 "R7" H 8070 2246 50  0000 L CNN
+F 1 "180R" H 8070 2155 50  0000 L CNN
+F 2 "" V 7930 2200 50  0000 C CNN
+F 3 "" H 8000 2200 50  0000 C CNN
+	1    8000 2200
 	1    0    0    -1
 $EndComp
@@
 L 0EsseivaN_Lib:R R8
 U 1 1 5CB800DB
-P 8250 1950
-F 0 "R8" H 8320 1996 50  0000 L CNN
-F 1 "560R" H 8320 1905 50  0000 L CNN
-F 2 "" V 8180 1950 50  0000 C CNN
-F 3 "" H 8250 1950 50  0000 C CNN
-	1    8250 1950
+P 8250 2200
+F 0 "R8" H 8320 2246 50  0000 L CNN
+F 1 "270R" H 8320 2155 50  0000 L CNN
+F 2 "" V 8180 2200 50  0000 C CNN
+F 3 "" H 8250 2200 50  0000 C CNN
+	1    8250 2200
 	1    0    0    -1
 $EndComp
@@
 L 0EsseivaN_Lib:R R6
 U 1 1 5CB8029A
-P 7550 1950
-F 0 "R6" H 7620 1996 50  0000 L CNN
-F 1 "560R" H 7620 1905 50  0000 L CNN
-F 2 "" V 7480 1950 50  0000 C CNN
-F 3 "" H 7550 1950 50  0000 C CNN
-	1    7550 1950
-	1    0    0    -1
-$EndComp
-Wire Wire Line
-	7550 2150 7550 2200
-Wire Wire Line
-	7900 2150 7900 2200
-Wire Wire Line
-	8250 2150 8250 2200
-Wire Wire Line
-	7550 1750 7550 1650
-Wire Wire Line
-	7550 1650 7900 1650
-Wire Wire Line
-	8250 1650 8250 1750
-Wire Wire Line
-	7900 1750 7900 1650
-Connection ~ 7900 1650
-Wire Wire Line
-	7900 1650 8250 1650
-Wire Wire Line
-	7900 1650 7900 1550
+P 7750 2200
+F 0 "R6" H 7681 2246 50  0000 R CNN
+F 1 "180R" H 7681 2155 50  0000 R CNN
+F 2 "" V 7680 2200 50  0000 C CNN
+F 3 "" H 7750 2200 50  0000 C CNN
+	1    7750 2200
+	1    0    0    -1
+$EndComp
 $Comp
 L 0EsseivaN_Lib:5V #PWR0124
 U 1 1 5CBB4994
-P 7900 1550
-F 0 "#PWR0124" H 7900 1400 50  0001 C CNN
-F 1 "5V" H 7917 1720 45  0000 C CNN
-F 2 "" H 7900 1550 50  0000 C CNN
-F 3 "" H 7900 1550 50  0000 C CNN
-	1    7900 1550
-	1    0    0    -1
-$EndComp
-Wire Wire Line
-	7550 2400 7550 3650
+P 8500 1300
+F 0 "#PWR0124" H 8500 1150 50  0001 C CNN
+F 1 "5V" H 8517 1470 45  0000 C CNN
+F 2 "" H 8500 1300 50  0000 C CNN
+F 3 "" H 8500 1300 50  0000 C CNN
+	1    8500 1300
+	1    0    0    -1
+$EndComp
 Wire Wire Line
 	7550 3650 7150 3650
@@
 L 0EsseivaN_Lib:5V #PWR0128
 U 1 1 5CD236ED
-P 10250 5750
-F 0 "#PWR0128" H 10250 5600 50  0001 C CNN
-F 1 "5V" H 10267 5920 45  0000 C CNN
-F 2 "" H 10250 5750 50  0000 C CNN
-F 3 "" H 10250 5750 50  0000 C CNN
-	1    10250 5750
-	1    0    0    -1
-$EndComp
-Wire Wire Line
-	10250 5750 10250 5850
+P 10000 5750
+F 0 "#PWR0128" H 10000 5600 50  0001 C CNN
+F 1 "5V" H 10017 5920 45  0000 C CNN
+F 2 "" H 10000 5750 50  0000 C CNN
+F 3 "" H 10000 5750 50  0000 C CNN
+	1    10000 5750
+	1    0    0    -1
+$EndComp
+Wire Wire Line
+	10000 5750 10000 5850
 $Comp
 L 0EsseivaN_Lib:3V3 #PWR0129
 U 1 1 5CD236F8
-P 10150 5750
-F 0 "#PWR0129" H 10150 5600 50  0001 C CNN
-F 1 "3V3" H 10168 5920 45  0000 C CNN
-F 2 "" H 10150 5750 50  0000 C CNN
-F 3 "" H 10150 5750 50  0000 C CNN
-	1    10150 5750
+P 9850 5750
+F 0 "#PWR0129" H 9850 5600 50  0001 C CNN
+F 1 "3V3" H 9868 5920 45  0000 C CNN
+F 2 "" H 9850 5750 50  0000 C CNN
+F 3 "" H 9850 5750 50  0000 C CNN
+	1    9850 5750
 	-1   0    0    -1
 $EndComp
 Wire Wire Line
-	10150 5750 10150 6050
-Wire Wire Line
-	10650 5850 10250 5850
-Connection ~ 10250 5850
-Wire Wire Line
-	10250 5850 10250 5950
-Wire Wire Line
-	10250 5950 10650 5950
-Wire Wire Line
-	10150 6050 10650 6050
-Wire Wire Line
-	10650 6150 10150 6150
-Wire Wire Line
-	10150 6150 10150 6050
-Connection ~ 10150 6050
+	9850 5750 9850 6050
+Wire Wire Line
+	10650 5850 10000 5850
+Connection ~ 10000 5850
+Wire Wire Line
+	10000 5850 10000 5950
+Wire Wire Line
+	10000 5950 10650 5950
+Wire Wire Line
+	9850 6050 10650 6050
+Wire Wire Line
+	10650 6150 9850 6150
+Wire Wire Line
+	9850 6150 9850 6050
+Connection ~ 9850 6050
 $Comp
 L 0EsseivaN_Lib:GND #PWR0130
@@
 P 6350 4750
 F 0 "U4" H 6950 6200 50  0000 C CNN
-F 1 "PIC18F45K40_44" H 6850 6100 50  0000 C CNN
+F 1 "PIC18F46K40_44" H 6850 6100 50  0000 C CNN
 F 2 "" H 6350 5050 50  0001 C CNN
 F 3 "https://www.digikey.ch/product-detail/en/microchip-technology/PIC18F45K40-I-PT/PIC18F45K40-I-PT-ND/6208274" H 6350 5050 50  0001 C CNN
@@
 	7600 3750 7600 2500
 Wire Wire Line
-	7600 2500 7900 2500
-Wire Wire Line
-	7900 2500 7900 2400
+	7600 2500 8000 2500
+Wire Wire Line
+	8000 2500 8000 2400
 Wire Wire Line
 	7150 3850 7650 3850
@@
 NoConn ~ 1150 2650
 NoConn ~ 1150 2750
-Text Notes 5400 2700 0    50   ~ 0
+Text Notes 3150 2000 0    50   ~ 0
 WARNING : Power MCP2210 and\nPIC with same voltages
 $Comp
@@
 Wire Wire Line
 	8650 5450 8750 5450
-$Comp
-L 0EsseivaN_Lib:5V #PWR0136
-U 1 1 5D02943E
-P 9800 5400
-F 0 "#PWR0136" H 9800 5250 50  0001 C CNN
-F 1 "5V" H 9888 5437 45  0000 L CNN
-F 2 "" H 9800 5400 50  0000 C CNN
-F 3 "" H 9800 5400 50  0000 C CNN
-	1    9800 5400
-	1    0    0    -1
-$EndComp
-Wire Wire Line
-	9800 5400 9800 5450
-Wire Wire Line
-	9800 5450 9700 5450
 Wire Wire Line
 	10650 3950 7900 3950
@@
 Text Label 7200 4550 0    50   ~ 0
 D4
+Text Label 7200 4350 0    50   ~ 0
+D3
+Text Label 7200 4250 0    50   ~ 0
+D2
+Text Label 7200 4150 0    50   ~ 0
+D1
+Text Label 7900 4050 0    50   ~ 0
+CLK
+Text Label 7900 3950 0    50   ~ 0
+DAC1
+$Comp
+L 0EsseivaN_Lib:CONN_01X02 X5
+U 1 1 5CBFA677
+P 10850 5600
+F 0 "X5" H 10928 5641 50  0000 L CNN
+F 1 "EXTENDER_COM" H 10928 5550 50  0000 L CNN
+F 2 "" H 10850 5450 50  0000 C CNN
+F 3 "" H 10700 5400 50  0000 C CNN
+	1    10850 5600
+	1    0    0    -1
+$EndComp
+Wire Wire Line
+	10550 5600 10250 5600
+Wire Wire Line
+	10250 5600 10250 5450
+Wire Wire Line
+	10250 5450 10150 5450
+Text Label 9750 5450 0    50   ~ 0
+COM
+$Comp
+L 0EsseivaN_Lib:LED_RGB P2
+U 1 1 5CC311F2
+P 8100 1750
+F 0 "P2" V 7922 2194 60  0000 L CNN
+F 1 "150141M173100" V 8028 2194 60  0000 L CNN
+F 2 "" H 8100 1900 60  0000 C CNN
+F 3 "" H 8100 1900 60  0000 C CNN
+	1    8100 1750
+	0    1    1    0
+$EndComp
+Wire Wire Line
+	7550 2450 7750 2450
+Wire Wire Line
+	7750 2450 7750 2400
+Wire Wire Line
+	7550 2450 7550 3650
+Wire Wire Line
+	7750 2000 7750 1900
+Wire Wire Line
+	8000 1900 8000 2000
+Wire Wire Line
+	8250 2000 8250 1900
+Wire Wire Line
+	8500 1300 8500 1350
+Wire Wire Line
+	10550 5600 10550 5500
+Wire Wire Line
+	10550 5500 10650 5500
+Wire Wire Line
+	10550 5600 10550 5700
+Wire Wire Line
+	10550 5700 10650 5700
 Wire Bus Line
 	1850 4500 4200 4500
@@
 Wire Bus Line
 	4600 4250 4600 6700
-Text Label 7200 4350 0    50   ~ 0
-D3
-Text Label 7200 4250 0    50   ~ 0
-D2
-Text Label 7200 4150 0    50   ~ 0
-D1
-Text Label 7900 4050 0    50   ~ 0
-CLK
-Text Label 7900 3950 0    50   ~ 0
-DAC1
+Connection ~ 10550 5600
+$Comp
+L 0EsseivaN_Lib:CAPA C9
+U 1 1 5CE24849
+P 10150 5550
+F 0 "C9" V 10250 5650 60  0000 L CNN
+F 1 "100nF" V 10350 5600 60  0000 L CNN
+F 2 "" H 10150 5550 60  0000 C CNN
+F 3 "" H 10150 5550 60  0000 C CNN
+	1    10150 5550
+	0    1    1    0
+$EndComp
+Connection ~ 10150 5450
+Wire Wire Line
+	10150 5450 9700 5450
+$Comp
+L 0EsseivaN_Lib:GND #PWR02
+U 1 1 5CE26235
+P 10150 5650
+F 0 "#PWR02" H 10150 5350 50  0001 C CNN
+F 1 "GND" H 10150 5450 50  0001 C CNN
+F 2 "" H 10150 5650 50  0000 C CNN
+F 3 "" H 10150 5650 50  0000 C CNN
+	1    10150 5650
+	1    0    0    -1
+$EndComp
 $EndSCHEMATC

Commit message: v0 Completed
Parts:
- C1, C4, C5, C7: footprint (none) -> 0EsseivaN_Lib:C_0805_HandSoldering
- C2: footprint (none) -> 0EsseivaN_Lib:CP_Radial_D5.0mm_P2.00mm
- C3, C6, C8, C9: footprint (none) -> 0EsseivaN_Lib:C_1206_HandSoldering
- F1: footprint (none) -> 0EsseivaN_Lib:Fuse_SMD1206_HandSoldering
- J1: footprint (none) -> 0EsseivaN_Lib:micro_usb
- J2: footprint (none) -> 0EsseivaN_Lib:Pin_Header_Straight_1x08_Pitch2.54mm
- J3, J4, J5: footprint (none) -> 0EsseivaN_Lib:CH_05P
- P1: footprint (none) -> 0EsseivaN_Lib:D_0603_HandSoldering
- P2: footprint (none) -> 0EsseivaN_Lib:LED_RGB_1411
- R1, R10, R11, R2, R3, R4, R5, R6, R7, R8, R9: footprint (none) -> 0EsseivaN_Lib:R_0603_HandSoldering
- SW1: footprint (none) -> 0EsseivaN_Lib:SLB12814
- U1: footprint (none) -> 0EsseivaN_Lib:MRF89XAM8A
- U2: footprint (none) -> 0EsseivaN_Lib:SOT-23-5_HandSoldering
- U3: footprint Housings_SSOP:SSOP-20_5.3x7.2mm_Pitch0.65mm -> 0EsseivaN_Lib:SSOP-20_5.3x7.2mm_Pitch0.65mm
- U4: footprint (none) -> 0EsseivaN_Lib:TQFP-44_10x10mm_Pitch0.8mm
- U5: footprint (none) -> 0EsseivaN_Lib:SOIC-16_3.9x9.9mm_Pitch1.27mm
- X1: footprint (none) -> 0EsseivaN_Lib:CH_07P
- X2, X3: footprint (none) -> 0EsseivaN_Lib:CH_08P
- X4: footprint (none) -> 0EsseivaN_Lib:CH_06P
- X5: footprint (none) -> 0EsseivaN_Lib:CH_02P
- Y1: footprint (none) -> 0EsseivaN_Lib:Oscillator_SMD_4pin_2.5x2.0mm_HandSoldering
Connections:
- net GND: now also X3.1 (P1); no longer X3.8 (P8)
- net P1: now also U5.10 (O7), X3.2 (P2); no longer U5.16 (O1), X3.1 (P1)
- net P2: now also U5.11 (O6), X3.3 (P3); no longer U5.15 (O2), X3.2 (P2)
- net P3: now also U5.12 (O5), X3.4 (P4); no longer U5.14 (O3), X3.3 (P3)
- net P4: now also X3.5 (P5); no longer X3.4 (P4)
- net P5: now also U5.14 (O3), X3.6 (P6); no longer U5.12 (O5), X3.5 (P5)
- net P6: now also U5.15 (O2), X3.7 (P7); no longer U5.11 (O6), X3.6 (P6)
- net P7: now also U5.16 (O1), X3.8 (P8); no longer U5.10 (O7), X3.7 (P7)
Other:
- note removed: "Ajouter led"

Commit message: v1
selectable mcu & rf transceiver power voltage
Parts:
- added X6: MCU_POWER_SELECT, 0EsseivaN_Lib:Pin_Header_Straight_1x03_Pitch2.54mm, symbol 0EsseivaN_Lib:CONN_01X03
- X4: footprint 0EsseivaN_Lib:CH_06P -> 0EsseivaN_Lib:CH_08P; symbol 0EsseivaN_Lib:CONN_01X06 -> 0EsseivaN_Lib:CONN_01X08
Connections:
- net 3V3: now also X6.1 (P1)
- net 5V: now also X6.3 (P3); no longer C5.2, C8.1, R4.2, U3.1 (Vdd), U4.28 (VDD), U4.7 (VDD)
- net GND: now also X4.7 (P7), X4.8 (P8); no longer X4.5 (P5), X4.6 (P6)
- new net VCC: C5.2, C8.1, R4.2, U3.1 (Vdd), U4.28 (VDD), U4.7 (VDD), X4.5 (P5), X4.6 (P6), X6.2 (P2)
Changed lines of the file:
@@
-	1    0    0    -1
-$EndComp
-$Comp
-L 0EsseivaN_Lib:5V #PWR0116
-U 1 1 5CBEEF46
-P 2150 2300
-F 0 "#PWR0116" H 2150 2150 50  0001 C CNN
-F 1 "5V" H 2097 2337 45  0000 R CNN
-F 2 "" H 2150 2300 50  0000 C CNN
-F 3 "" H 2150 2300 50  0000 C CNN
-	1    2150 2300
 	1    0    0    -1
 $EndComp
@@
 Text Label 4300 3950 0    50   ~ 0
 ~LOWPWR
-$Comp
-L 0EsseivaN_Lib:5V #PWR0104
-U 1 1 5CC49943
-P 6600 3050
-F 0 "#PWR0104" H 6600 2900 50  0001 C CNN
-F 1 "5V" H 6617 3220 45  0000 C CNN
-F 2 "" H 6600 3050 50  0000 C CNN
-F 3 "" H 6600 3050 50  0000 C CNN
-	1    6600 3050
-	1    0    0    -1
-$EndComp
 Connection ~ 6600 3050
 $Comp
@@
 	3600 2100 3600 2150
 Connection ~ 3050 2100
-$Comp
-L 0EsseivaN_Lib:5V #PWR0122
-U 1 1 5CE9F6D1
-P 3050 2050
-F 0 "#PWR0122" H 3050 1900 50  0001 C CNN
-F 1 "5V" H 3067 2220 45  0000 C CNN
-F 2 "" H 3050 2050 50  0000 C CNN
-F 3 "" H 3050 2050 50  0000 C CNN
-	1    3050 2050
-	1    0    0    -1
-$EndComp
 Wire Wire Line
 	3050 2050 3050 2100
@@
 	10400 5350 10650 5350
 $Comp
-L 0EsseivaN_Lib:CONN_01X06 X4
+L 0EsseivaN_Lib:CONN_01X08 X4
 U 1 1 5CD219E8
-P 10850 6150
-F 0 "X4" H 10928 6241 50  0000 L CNN
-F 1 "EXTENDER_POWER_1" H 10928 6150 50  0000 L CNN
-F 2 "0EsseivaN_Lib:CH_06P" H 10850 6150 50  0001 C CNN
-F 3 "" H 10850 6150 50  0000 C CNN
-	1    10850 6150
+P 9650 3250
+F 0 "X4" H 9728 3341 50  0000 L CNN
+F 1 "EXTENDER_POWER_1" H 9728 3250 50  0000 L CNN
+F 2 "0EsseivaN_Lib:CH_08P" H 9650 3250 50  0001 C CNN
+F 3 "" H 9650 3250 50  0000 C CNN
+	1    9650 3250
 	1    0    0    -1
 $EndComp
@@
 L 0EsseivaN_Lib:5V #PWR0128
 U 1 1 5CD236ED
-P 10000 5750
-F 0 "#PWR0128" H 10000 5600 50  0001 C CNN
-F 1 "5V" H 10017 5920 45  0000 C CNN
-F 2 "" H 10000 5750 50  0000 C CNN
-F 3 "" H 10000 5750 50  0000 C CNN
-	1    10000 5750
-	1    0    0    -1
-$EndComp
-Wire Wire Line
-	10000 5750 10000 5850
+P 8800 2800
+F 0 "#PWR0128" H 8800 2650 50  0001 C CNN
+F 1 "5V" H 8817 2970 45  0000 C CNN
+F 2 "" H 8800 2800 50  0000 C CNN
+F 3 "" H 8800 2800 50  0000 C CNN
+	1    8800 2800
+	1    0    0    -1
+$EndComp
+Wire Wire Line
+	8800 2800 8800 2900
 $Comp
 L 0EsseivaN_Lib:3V3 #PWR0129
 U 1 1 5CD236F8
-P 9850 5750
-F 0 "#PWR0129" H 9850 5600 50  0001 C CNN
-F 1 "3V3" H 9868 5920 45  0000 C CNN
-F 2 "" H 9850 5750 50  0000 C CNN
-F 3 "" H 9850 5750 50  0000 C CNN
-	1    9850 5750
+P 8650 2800
+F 0 "#PWR0129" H 8650 2650 50  0001 C CNN
+F 1 "3V3" H 8668 2970 45  0000 C CNN
+F 2 "" H 8650 2800 50  0000 C CNN
+F 3 "" H 8650 2800 50  0000 C CNN
+	1    8650 2800
 	-1   0    0    -1
 $EndComp
 Wire Wire Line
-	9850 5750 9850 6050
-Wire Wire Line
-	10650 5850 10000 5850
-Connection ~ 10000 5850
-Wire Wire Line
-	10000 5850 10000 5950
-Wire Wire Line
-	10000 5950 10650 5950
-Wire Wire Line
-	9850 6050 10650 6050
-Wire Wire Line
-	10650 6150 9850 6150
-Wire Wire Line
-	9850 6150 9850 6050
-Connection ~ 9850 6050
+	8650 2800 8650 3100
+Wire Wire Line
+	9450 2900 8800 2900
+Connection ~ 8800 2900
+Wire Wire Line
+	8800 2900 8800 3000
+Wire Wire Line
+	8800 3000 9450 3000
+Wire Wire Line
+	8650 3100 9450 3100
+Wire Wire Line
+	9450 3200 8650 3200
+Wire Wire Line
+	8650 3200 8650 3100
+Connection ~ 8650 3100
 $Comp
 L 0EsseivaN_Lib:GND #PWR0130
 U 1 1 5CD66E90
-P 10250 6450
-F 0 "#PWR0130" H 10250 6150 50  0001 C CNN
-F 1 "GND" H 10250 6250 50  0001 C CNN
-F 2 "" H 10250 6450 50  0000 C CNN
-F 3 "" H 10250 6450 50  0000 C CNN
-	1    10250 6450
-	1    0    0    -1
-$EndComp
-Wire Wire Line
-	10250 6450 10250 6350
-Wire Wire Line
-	10250 6250 10650 6250
-Wire Wire Line
-	10650 6350 10250 6350
-Connection ~ 10250 6350
-Wire Wire Line
-	10250 6350 10250 6250
+P 9050 3700
+F 0 "#PWR0130" H 9050 3400 50  0001 C CNN
+F 1 "GND" H 9050 3500 50  0001 C CNN
+F 2 "" H 9050 3700 50  0000 C CNN
+F 3 "" H 9050 3700 50  0000 C CNN
+	1    9050 3700
+	1    0    0    -1
+$EndComp
+Wire Wire Line
+	9050 3700 9050 3600
+Wire Wire Line
+	9050 3500 9450 3500
+Wire Wire Line
+	9450 3600 9050 3600
+Connection ~ 9050 3600
+Wire Wire Line
+	9050 3600 9050 3500
 $Comp
 L 0EsseivaN_Lib:GND #PWR0131
@@
 Text Label 10600 4150 2    50   ~ 0
 D1
-Text Label 10600 5850 2    50   ~ 0
+Text Label 9400 2900 2    50   ~ 0
 5V
-Text Label 10600 5950 2    50   ~ 0
+Text Label 9400 3000 2    50   ~ 0
 5V
-Text Label 10600 6050 2    50   ~ 0
+Text Label 9400 3100 2    50   ~ 0
 3V3
-Text Label 10600 6150 2    50   ~ 0
+Text Label 9400 3200 2    50   ~ 0
 3V3
-Text Label 10600 6250 2    50   ~ 0
+Text Label 9400 3500 2    50   ~ 0
 GND
-Text Label 10600 6350 2    50   ~ 0
+Text Label 9400 3600 2    50   ~ 0
 GND
 Text Label 7200 5450 0    50   ~ 0
@@
 Wire Wire Line
 	3400 900  3300 900
+$Comp
+L 0EsseivaN_Lib:CONN_01X03 X6
+U 1 1 5CD3DBAD
+P 5450 950
+F 0 "X6" H 5367 1273 50  0000 C CNN
+F 1 "MCU_POWER_SELECT" H 5367 1364 50  0000 C CNN
+F 2 "0EsseivaN_Lib:Pin_Header_Straight_1x03_Pitch2.54mm" H 5367 817 50  0001 C CNN
+F 3 "" H 5300 750 50  0000 C CNN
+	1    5450 950
+	-1   0    0    1
+$EndComp
+$Comp
+L 0EsseivaN_Lib:5V #PWR0136
+U 1 1 5CD3EE7C
+P 5850 900
+F 0 "#PWR0136" H 5850 750 50  0001 C CNN
+F 1 "5V" H 5867 1070 45  0000 C CNN
+F 2 "" H 5850 900 50  0000 C CNN
+F 3 "" H 5850 900 50  0000 C CNN
+	1    5850 900
+	1    0    0    -1
+$EndComp
+$Comp
+L 0EsseivaN_Lib:3V3 #PWR0137
+U 1 1 5CD3F192
+P 6150 900
+F 0 "#PWR0137" H 6150 750 50  0001 C CNN
+F 1 "3V3" H 6167 1070 45  0000 C CNN
+F 2 "" H 6150 900 50  0000 C CNN
+F 3 "" H 6150 900 50  0000 C CNN
+	1    6150 900
+	1    0    0    -1
+$EndComp
+Wire Wire Line
+	5850 900  5850 950
+Wire Wire Line
+	5850 950  5650 950
+Wire Wire Line
+	5650 1150 6150 1150
+Wire Wire Line
+	6150 1150 6150 900
+$Comp
+L 0EsseivaN_Lib:VCC #PWR0138
+U 1 1 5CD8ED8A
+P 6000 900
+F 0 "#PWR0138" H 6000 750 50  0001 C CNN
+F 1 "VCC" H 6017 1073 50  0000 C CNN
+F 2 "" H 6000 900 50  0000 C CNN
+F 3 "" H 6000 900 50  0000 C CNN
+	1    6000 900
+	1    0    0    -1
+$EndComp
+Wire Wire Line
+	6000 900  6000 1050
+Wire Wire Line
+	6000 1050 5650 1050
+$Comp
+L 0EsseivaN_Lib:VCC #PWR0104
+U 1 1 5CDA78CE
+P 3050 2050
+F 0 "#PWR0104" H 3050 1900 50  0001 C CNN
+F 1 "VCC" H 3067 2223 50  0000 C CNN
+F 2 "" H 3050 2050 50  0000 C CNN
+F 3 "" H 3050 2050 50  0000 C CNN
+	1    3050 2050
+	1    0    0    -1
+$EndComp
+$Comp
+L 0EsseivaN_Lib:5V #PWR0116
+U 1 1 5CBEEF46
+P 2150 2300
+F 0 "#PWR0116" H 2150 2150 50  0001 C CNN
+F 1 "5V" H 2097 2337 45  0000 R CNN
+F 2 "" H 2150 2300 50  0000 C CNN
+F 3 "" H 2150 2300 50  0000 C CNN
+	1    2150 2300
+	1    0    0    -1
+$EndComp
+$Comp
+L 0EsseivaN_Lib:VCC #PWR0122
+U 1 1 5CDA9820
+P 6600 3050
+F 0 "#PWR0122" H 6600 2900 50  0001 C CNN
+F 1 "VCC" H 6617 3223 50  0000 C CNN
+F 2 "" H 6600 3050 50  0000 C CNN
+F 3 "" H 6600 3050 50  0000 C CNN
+	1    6600 3050
+	1    0    0    -1
+$EndComp
+$Comp
+L 0EsseivaN_Lib:VCC #PWR0139
+U 1 1 5CDA9D2E
+P 8500 2800
+F 0 "#PWR0139" H 8500 2650 50  0001 C CNN
+F 1 "VCC" H 8447 2837 50  0000 R CNN
+F 2 "" H 8500 2800 50  0000 C CNN
+F 3 "" H 8500 2800 50  0000 C CNN
+	1    8500 2800
+	1    0    0    -1
+$EndComp
+Wire Wire Line
+	8500 2800 8500 3300
+Wire Wire Line
+	8500 3300 9450 3300
+Wire Wire Line
+	9450 3400 8500 3400
+Wire Wire Line
+	8500 3400 8500 3300
+Connection ~ 8500 3300
+Text Label 9400 3300 2    50   ~ 0
+VCC
+Text Label 9400 3400 2    50   ~ 0
+VCC
+$Comp
+L power:PWR_FLAG #FLG0102
+U 1 1 5CE6BEF9
+P 6350 900
+F 0 "#FLG0102" H 6350 975 50  0001 C CNN
+F 1 "PWR_FLAG" H 6418 942 50  0000 L CNN
+F 2 "" H 6350 900 50  0001 C CNN
+F 3 "~" H 6350 900 50  0001 C CNN
+	1    6350 900
+	1    0    0    -1
+$EndComp
+Wire Wire Line
+	6350 900  6350 1050
+Wire Wire Line
+	6350 1050 6000 1050
 Wire Bus Line
 	1850 4500 4200 4500
@@
 Wire Bus Line
 	4600 4250 4600 6700
+Connection ~ 6000 1050
 $EndSCHEMATC
