File: Hardware/USB_Tool.sch (KiCad schematic (older format))
At the start: 45 parts, among them J1 USB_B_Micro, J2 CONN_ICSP, P1 TLMS1000, P2 150141M173100, P3 Green, P4 Green, SW1 SW_2TO1, U1 MRF89XAM8A, U2 NCP114, U3 MCP2210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

Commit message: v4 updated
Parts:
- removed C4: 1uF, 0EsseivaN_Lib:C_0805_HandSoldering, symbol 0EsseivaN_Lib:CAPA_P
- removed U3: MCP2210, 0EsseivaN_Lib:SSOP-20_5.3x7.2mm_Pitch0.65mm, symbol 0EsseivaN_Lib:MCP2210
- removed X9: Extender_I2C_3, 0EsseivaN_Lib:CH_02P, symbol 0EsseivaN_Lib:CONN_01X02
- removed Y1: DSC6003JI2A, 0EsseivaN_Lib:Oscillator_SMD_4pin_2.5x2.0mm_HandSoldering, symbol 0EsseivaN_Lib:DSC6003JI2A
- added P1: RED, 0EsseivaN_Lib:D_0603_HandSoldering, symbol 0EsseivaN_Lib:LED
- added P5: Blue, 0EsseivaN_Lib:D_0805_HandSoldering, symbol 0EsseivaN_Lib:LED
- added P6, P7: Green, 0EsseivaN_Lib:D_0603_HandSoldering, symbol 0EsseivaN_Lib:LED
- added R16: 120R, 0EsseivaN_Lib:R_0603_HandSoldering, symbol 0EsseivaN_Lib:R
- added R17: 270R, 0EsseivaN_Lib:R_0603_HandSoldering, symbol 0EsseivaN_Lib:R
- added R18: 150R, 0EsseivaN_Lib:R_0603_HandSoldering, symbol 0EsseivaN_Lib:R
- added R19, R20, R21, R22, R23: 4k7, 0EsseivaN_Lib:R_0603_HandSoldering, symbol 0EsseivaN_Lib:R
- added U3: MCP2221A, 0EsseivaN_Lib:TSSOP-14_4.4x5mm_Pitch0.65mm, symbol 0EsseivaN_Lib:MCP2221A
- added X10, X9: Extension, 0EsseivaN_Lib:Pin_Header_Straight_1x09_Pitch2.54mm, symbol 0EsseivaN_Lib:CONN_01X09
- added X11: EXTENDER_LED_1, 0EsseivaN_Lib:CH_02P, symbol 0EsseivaN_Lib:CONN_01X02
- C5: value 470nF -> 100nF; footprint 0EsseivaN_Lib:C_0805_HandSoldering -> 0EsseivaN_Lib:C_1206_HandSoldering
- C6: footprint 0EsseivaN_Lib:C_1206_HandSoldering -> 0EsseivaN_Lib:C_0805_HandSoldering
- P2: value 150141M173100 -> RGB
- P8: renamed from P1; value TLMS1000 -> Blue; footprint 0EsseivaN_Lib:D_0603_HandSoldering -> 0EsseivaN_Lib:D_0805_HandSoldering
- R10, R12, R13, R5, R9: value 1k -> 4k7
- R3: value 1k -> 150R
- R6, R7: value 180R -> 330R
- R8: value 270R -> 560R
- X1: footprint 0EsseivaN_Lib:CH_04P -> 0EsseivaN_Lib:CH_03P; symbol 0EsseivaN_Lib:CONN_01X04 -> 0EsseivaN_Lib:CONN_01X03
- X12: renamed from J2; footprint 0EsseivaN_Lib:Pin_Header_Straight_1x08_Pitch2.54mm -> 0EsseivaN_Lib:Pin_Header_Straight_1x05_Pitch2.54mm
- X2: value EXTENDER_IO_1 -> EXTENDER_IO_2
- X3: value EXTENDER_IO_2 -> EXTENDER_IO_1; footprint 0EsseivaN_Lib:CH_08P -> 0EsseivaN_Lib:CH_06P; symbol 0EsseivaN_Lib:CONN_01X08 -> 0EsseivaN_Lib:CONN_01X06
- X5: value EXTENDER_POWER_2 -> EXTENDER_POWER_1
- renumbered X7 to X6, X8 to X7
Connections:
- net labels added: CLKR, D0, DAC_OUT, ICSP_VCC, LED0, LED1, LED2, LEDRGB_B, LEDRGB_G, LEDRGB_R, Rx, SSPND, Tx, USBCFG, USB_IOC, ~INT0, ~INT1, ~INT2, ~MCLR, ~RESET_USB
- net labels removed: BRA, BRR, CLK, CS_EXT, D10, D11, D6, D7, D8, D9, INT, LED_B, LED_G, LED_R, RESET_USB, SPI_LED, VPP, ~LOWPWR, ~SSPND, ~USBCFG
- wire segments 226 -> 323
- no-connect marks 12 -> 6
Other:
- note added: "3V3"
- note added: "40mm separation"
- note added: "5V"
- note added: "CLKR"
- note added: "DAC_OUT"
- note added: "GND"
- note added: "LED0"
- note added: "LED1"
- note added: "SCL"
- note added: "SDA"
- note removed: "12MHz\noscillator"
- note removed: "USB to SPI"
- moved on the sheet: C1, C2, C5, C6, C7, C9, F1, J1, P2, P3, P4, P8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

Commit message: v4 final
Parts:
- F1: value 500mA -> 250mA
Changed lines of the file:
@@
 P 2650 950
 F 0 "F1" V 2453 950 50  0000 C CNN
-F 1 "500mA" V 2544 950 50  0000 C CNN
+F 1 "250mA" V 2544 950 50  0000 C CNN
 F 2 "0EsseivaN_Lib:Fuse_SMD2410_HandSoldering" V 2580 950 50  0001 C CNN
 F 3 "" H 2650 950 50  0000 C CNN

Commit message: 1
Parts:
- removed C3: 100nF, 0EsseivaN_Lib:C_1206_HandSoldering, symbol 0EsseivaN_Lib:CAPA
- removed C6: 4.7uF, 0EsseivaN_Lib:C_0805_HandSoldering, symbol 0EsseivaN_Lib:CAPA
- removed R10, R5, R9: 4k7, 0EsseivaN_Lib:R_0603_HandSoldering, symbol 0EsseivaN_Lib:R
- removed U1: MRF89XAM8A, 0EsseivaN_Lib:MRF89XAM8A, symbol 0EsseivaN_Lib:MRF89XAM8A
- removed X1: EXTENDER_SPI_1, 0EsseivaN_Lib:CH_03P, symbol 0EsseivaN_Lib:CONN_01X03
- removed X10, X9: Extension, 0EsseivaN_Lib:Pin_Header_Straight_1x09_Pitch2.54mm, symbol 0EsseivaN_Lib:CONN_01X09
- removed X11: EXTENDER_LED_1, 0EsseivaN_Lib:CH_02P, symbol 0EsseivaN_Lib:CONN_01X02
- removed X2: EXTENDER_IO_2, 0EsseivaN_Lib:CH_05P, symbol 0EsseivaN_Lib:CONN_01X05
- removed X3: EXTENDER_IO_1, 0EsseivaN_Lib:CH_06P, symbol 0EsseivaN_Lib:CONN_01X06
- removed X4: EXTENDER_POWER_2, 0EsseivaN_Lib:CH_03P, symbol 0EsseivaN_Lib:CONN_01X03
- removed X5: EXTENDER_POWER_1, 0EsseivaN_Lib:CH_03P, symbol 0EsseivaN_Lib:CONN_01X03
- removed X6: Extender_I2C_1, 0EsseivaN_Lib:CH_02P, symbol 0EsseivaN_Lib:CONN_01X02
- removed X7: Extender_I2C_2, 0EsseivaN_Lib:CH_02P, symbol 0EsseivaN_Lib:CONN_01X02
- added J2, J3: EXT, symbol 0EsseivaN_Lib:Conn_02x08_Odd_Even
- R12, R13: value 4k7 -> 3k3
Connections:
- net labels added: D10, D11, D6, D7, D8, D9, EXT_LED_B, EXT_LED_G, TBD, ~INT3
- net labels removed: IRQ0, IRQ1, MISO, MOSI, RESET_RF, SCK, ~CSCON, ~CSDAT
- wire segments 323 -> 217
Other:
- note added: "50mm separation"
- note added: "EXTENSION BUS"
- note added: "USB BRIDGE BUS"
- note removed: "3V3"
- note removed: "40mm separation"
- note removed: "5V"
- note removed: "CLKR"
- note removed: "DAC_OUT"
- note removed: "GND"
- note removed: "LED0"
- note removed: "LED1"
- note removed: "SCL"
- note removed: "SDA"
- moved on the sheet: C2, C5, C7, C8, C9, F1, P1, P2, P3, P4, P5, P6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
