File: extensions/RF_433MHz_Receiver/Hardware/RF_433MHz_Receiver.kicad_pcb (KiCad board)
At the start: 2 copper layers, 55 x 40 mm, 17 parts, among them J1 CONN_ICSP, P1 1V8, U1 PIC16F15323, U2 RF_RECEIVER, X1 Extension_1, X2 Extension_2, X3 Extension, X4 Extension

Commit message: v4 final
Parts:
- X1, X2: moved to B.Cu
- turned X1 to 180 degrees
- turned X2 to 180 degrees
Other:
- board text added: "+"
- board text added: "EXT_RF_RX 24.06.19 - v00 EsseivaN"
- board text removed: "EXT_RF_RX 23.06.19 - v00 EsseivaN"
