File: extensions/RF_433MHz_Receiver/Hardware/RF_433MHz_Receiver.sch (KiCad schematic (older format))
At the start: 17 parts, among them J1 CONN_ICSP, P1 1V8, U1 PIC16F15323, U2 RF_RECEIVER, X1 Extension_1, X2 Extension_2, X3 Extension, X4 Extension

Commit message: v4 final
Changed lines of the file:
@@
 Sheet 1 1
 Title "RF_433MHz_Receiver"
-Date "2019-06-23"
+Date "2019-06-24"
 Rev "00"
 Comp "EsseivaN"
@@
 Comment4 ""
 $EndDescr
-Text Label 2700 4500 0    50   ~ 0
+Text Label 2700 4500 0    50   ~ 6
 SDA
-Text Label 2700 4600 0    50   ~ 0
+Text Label 2700 4600 0    50   ~ 6
 SCL
 $Comp
@@
 Wire Wire Line
 	2500 2700 2400 2700
-Text GLabel 3950 2600 0    50   BiDi ~ 0
+Text GLabel 3950 2600 0    50   BiDi ~ 6
 ICSPDAT
-Text GLabel 3950 2700 0    50   Input ~ 0
+Text GLabel 3950 2700 0    50   Input ~ 6
 ICSPCLK
-Text GLabel 3750 2900 0    50   UnSpc ~ 0
+Text GLabel 3750 2900 0    50   UnSpc ~ 6
 VPP
-Text GLabel 4750 2600 2    50   BiDi ~ 0
+Text GLabel 4750 2600 2    50   BiDi ~ 6
 SCL
-Text GLabel 4750 2700 2    50   BiDi ~ 0
+Text GLabel 4750 2700 2    50   BiDi ~ 6
 SDA
 Wire Wire Line
@@
 Wire Wire Line
 	4650 2700 4750 2700
-Text GLabel 3600 4050 0    50   BiDi ~ 0
+Text GLabel 3600 4050 0    50   BiDi ~ 6
 SCL
-Text GLabel 3600 4200 0    50   BiDi ~ 0
+Text GLabel 3600 4200 0    50   BiDi ~ 6
 SDA
 Wire Wire Line
@@
 Wire Wire Line
 	3950 2600 4050 2600
-Text GLabel 2700 2800 2    50   BiDi ~ 0
+Text GLabel 2700 2800 2    50   BiDi ~ 6
 ICSPDAT
-Text GLabel 2700 2900 2    50   Output ~ 0
+Text GLabel 2700 2900 2    50   Output ~ 6
 ICSPCLK
 Wire Wire Line
@@
 Wire Wire Line
 	2400 2800 2700 2800
-Text GLabel 2700 2500 2    50   UnSpc ~ 0
+Text GLabel 2700 2500 2    50   UnSpc ~ 6
 VPP
 Wire Wire Line
@@
 	0    1    1    0
 $EndComp
-Text Notes 5950 2800 0    50   ~ 0
+Text Notes 5950 2800 0    50   ~ 6
 R2..6\n5x1k
 Wire Wire Line
@@
 Wire Wire Line
 	3800 4600 2550 4600
-Text Label 2700 4400 0    50   ~ 0
+Text Label 2700 4400 0    50   ~ 6
 3V3
-Text Label 2700 4300 0    50   ~ 0
+Text Label 2700 4300 0    50   ~ 6
 5V
-Text Label 2700 5100 0    50   ~ 0
+Text Label 2700 5100 0    50   ~ 6
 GND
-Text Label 2700 4800 0    50   ~ 0
+Text Label 2700 4800 0    50   ~ 6
 DAC_OUT
-Text Label 2700 4700 0    50   ~ 0
+Text Label 2700 4700 0    50   ~ 6
 CLKR
 $Comp
@@
 Wire Wire Line
 	3100 5100 4250 5100
-Text Label 5200 4300 0    50   ~ 0
+Text Label 5200 4300 0    50   ~ 6
 D0
-Text Label 5200 4400 0    50   ~ 0
+Text Label 5200 4400 0    50   ~ 6
 D1
-Text Label 5200 4500 0    50   ~ 0
+Text Label 5200 4500 0    50   ~ 6
 D2
-Text Label 5200 4600 0    50   ~ 0
+Text Label 5200 4600 0    50   ~ 6
 D3
-Text Label 5200 4700 0    50   ~ 0
+Text Label 5200 4700 0    50   ~ 6
 D4
-Text Label 5200 4800 0    50   ~ 0
+Text Label 5200 4800 0    50   ~ 6
 D5
-Text Label 5200 5000 0    50   ~ 0
+Text Label 5200 5000 0    50   ~ 6
 ~INT1
-Text Label 5200 5100 0    50   ~ 0
+Text Label 5200 5100 0    50   ~ 6
 ~INT2
 Wire Wire Line
@@
 Wire Wire Line
 	5150 5100 6100 5100
-Text Notes 5150 5300 2    59   ~ 0
+Text Notes 5150 5300 2    59   ~ 6
 3V3 MAX !
-Text Notes 2550 5250 2    59   ~ 0
+Text Notes 2550 5250 2    59   ~ 6
 3V3 MAX !
 Wire Wire Line
@@
 Wire Wire Line
 	5150 4900 5500 4900
-Text Label 5200 4900 0    50   ~ 0
+Text Label 5200 4900 0    50   ~ 6
 ~INT0
 Wire Wire Line
